File: 9VReg.sch (KiCad schematic (older format))
At the start: 7 parts, among them J1 PWROUT, J2 PWRIN, U1 L7809

Commit message: 9VReg Mk. II
Parts:
- removed C2: 10u, Capacitors_THT:CP_Radial_D5.0mm_P2.50mm, symbol CP
- removed D1: LED, LEDs:LED_D3.0mm, symbol LED
- removed R1: 330, Resistors_THT:R_Axial_DIN0207_L6.3mm_D2.5mm_P10.16mm_Horizontal, symbol R
- added C?: 1000u, symbol CP
- added C? (x2): 470u, symbol CP
- added D?: LED, symbol LED
- added Q?: TIP35, symbol Q_NPN_BCE
- added Q?: BD139, symbol Q_NPN_ECB
- added R? (x2): 220, symbol R
- added R?: 12k, symbol R
- added R?: 330, symbol R
Connections:
- net GND: now also C?.2, C?.2, C?.2, D?.1 (K), R?.2
- net +9V: no longer names the net of U1.3 (OUT)
- net +9V: now also C?.1, Q?.2 (C), Q?.2 (C), R?.2; no longer J1.1 (Pin_1)
- new net: J1.1 (Pin_1), Q?.3 (E), R?.1
- new net: C?.1, R?.1, R?.2
- new net: C?.1, Q?.3 (B), R?.1, R?.1
- new net: Q?.1 (B), Q?.1 (E)
- new net: D?.2 (A), R?.2
Other:
- moved on the sheet: J1
Changed lines of the file:
@@
-$EndComp
-$Comp
-L LED D1
-U 1 1 5AF27C09
-P 6300 4550
-F 0 "D1" H 6300 4650 50  0000 C CNN
-F 1 "LED" H 6300 4450 50  0000 C CNN
-F 2 "LEDs:LED_D3.0mm" H 6300 4550 50  0001 C CNN
-F 3 "" H 6300 4550 50  0001 C CNN
-	1    6300 4550
-	0    -1   -1   0
-$EndComp
-$Comp
-L R R1
-U 1 1 5AF27CE3
-P 6300 4150
-F 0 "R1" V 6380 4150 50  0000 C CNN
-F 1 "330" V 6300 4150 50  0000 C CNN
-F 2 "Resistors_THT:R_Axial_DIN0207_L6.3mm_D2.5mm_P10.16mm_Horizontal" V 6230 4150 50  0001 C CNN
-F 3 "" H 6300 4150 50  0001 C CNN
-	1    6300 4150
-	1    0    0    -1
 $EndComp
 $Comp
@@
 $EndComp
 $Comp
-L GND #PWR02
-U 1 1 5AF27D98
-P 6300 4900
-F 0 "#PWR02" H 6300 4650 50  0001 C CNN
-F 1 "GND" H 6300 4750 50  0000 C CNN
-F 2 "" H 6300 4900 50  0001 C CNN
-F 3 "" H 6300 4900 50  0001 C CNN
-	1    6300 4900
-	1    0    0    -1
-$EndComp
-$Comp
 L Conn_01x02 J1
 U 1 1 5AF27DF6
-P 7200 3900
-F 0 "J1" H 7200 4000 50  0000 C CNN
-F 1 "PWROUT" H 7200 3700 50  0000 C CNN
-F 2 "TerminalBlocks_Phoenix:TerminalBlock_Phoenix_MKDS1.5-2pol" H 7200 3900 50  0001 C CNN
-F 3 "" H 7200 3900 50  0001 C CNN
-	1    7200 3900
-	1    0    0    -1
-$EndComp
-$Comp
-L GND #PWR03
-U 1 1 5AF27E29
-P 6900 4100
-F 0 "#PWR03" H 6900 3850 50  0001 C CNN
-F 1 "GND" H 6900 3950 50  0000 C CNN
-F 2 "" H 6900 4100 50  0001 C CNN
-F 3 "" H 6900 4100 50  0001 C CNN
-	1    6900 4100
-	1    0    0    -1
-$EndComp
-Connection ~ 6300 3900
-Wire Wire Line
-	6900 4000 7000 4000
-Wire Wire Line
-	6900 4100 6900 4000
-Wire Wire Line
-	6300 4700 6300 4900
-Wire Wire Line
-	6300 4300 6300 4400
-Wire Wire Line
-	6300 3900 6300 4000
-Wire Wire Line
-	6100 3900 7000 3900
-Connection ~ 5000 4100
-Wire Wire Line
-	5800 4200 5800 4400
-Wire Wire Line
-	5000 4100 4900 4100
-Wire Wire Line
-	5000 4000 5000 4400
-Wire Wire Line
-	4900 4000 5000 4000
-Wire Wire Line
-	4900 3900 5500 3900
+P 8800 3800
+F 0 "J1" H 8800 3900 50  0000 C CNN
+F 1 "PWROUT" H 8800 3600 50  0000 C CNN
+F 2 "TerminalBlocks_Phoenix:TerminalBlock_Phoenix_MKDS1.5-2pol" H 8800 3800 50  0001 C CNN
+F 3 "" H 8800 3800 50  0001 C CNN
+	1    8800 3800
+	1    0    0    -1
+$EndComp
 $Comp
 L CP C1
@@
 	1    0    0    -1
 $EndComp
-Wire Wire Line
-	5000 4400 5800 4400
-Wire Wire Line
-	5300 4300 5300 4500
-Wire Wire Line
-	5300 4000 5300 3900
-Connection ~ 5300 3900
-$Comp
-L CP C2
-U 1 1 5AF282F8
-P 6600 4550
-F 0 "C2" H 6625 4650 50  0000 L CNN
-F 1 "10u" H 6625 4450 50  0000 L CNN
-F 2 "Capacitors_THT:CP_Radial_D5.0mm_P2.50mm" H 6638 4400 50  0001 C CNN
-F 3 "" H 6600 4550 50  0001 C CNN
-	1    6600 4550
-	1    0    0    -1
-$EndComp
-Wire Wire Line
-	6600 4400 6600 3900
-Connection ~ 6600 3900
-Wire Wire Line
-	6600 4700 6600 4850
-Wire Wire Line
-	6600 4850 6300 4850
-Connection ~ 6300 4850
-Connection ~ 5300 4400
-$Comp
-L +9V #PWR04
-U 1 1 5AF28900
-P 6300 3900
-F 0 "#PWR04" H 6300 3750 50  0001 C CNN
-F 1 "+9V" H 6300 4040 50  0000 C CNN
-F 2 "" H 6300 3900 50  0001 C CNN
-F 3 "" H 6300 3900 50  0001 C CNN
-	1    6300 3900
-	1    0    0    -1
-$EndComp
 $Comp
 L +12V #PWR05
@@
 	1    0    0    -1
 $EndComp
+$Comp
+L CP C?
+U 1 1 5BBD88D8
+P 6200 4150
+F 0 "C?" H 6225 4250 50  0000 L CNN
+F 1 "1000u" H 6225 4050 50  0000 L CNN
+F 2 "" H 6238 4000 50  0001 C CNN
+F 3 "" H 6200 4150 50  0001 C CNN
+	1    6200 4150
+	1    0    0    -1
+$EndComp
+$Comp
+L CP C?
+U 1 1 5BBD8903
+P 6700 4150
+F 0 "C?" H 6725 4250 50  0000 L CNN
+F 1 "470u" H 6725 4050 50  0000 L CNN
+F 2 "" H 6738 4000 50  0001 C CNN
+F 3 "" H 6700 4150 50  0001 C CNN
+	1    6700 4150
+	1    0    0    -1
+$EndComp
+$Comp
+L CP C?
+U 1 1 5BBD8938
+P 7200 4150
+F 0 "C?" H 7225 4250 50  0000 L CNN
+F 1 "470u" H 7225 4050 50  0000 L CNN
+F 2 "" H 7238 4000 50  0001 C CNN
+F 3 "" H 7200 4150 50  0001 C CNN
+	1    7200 4150
+	1    0    0    -1
+$EndComp
+$Comp
+L R R?
+U 1 1 5BBD89EA
+P 6450 3900
+F 0 "R?" V 6530 3900 50  0000 C CNN
+F 1 "220" V 6450 3900 50  0000 C CNN
+F 2 "" V 6380 3900 50  0001 C CNN
+F 3 "" H 6450 3900 50  0001 C CNN
+	1    6450 3900
+	0    1    1    0
+$EndComp
+$Comp
+L R R?
+U 1 1 5BBD8A39
+P 6950 3900
+F 0 "R?" V 7030 3900 50  0000 C CNN
+F 1 "220" V 6950 3900 50  0000 C CNN
+F 2 "" V 6880 3900 50  0001 C CNN
+F 3 "" H 6950 3900 50  0001 C CNN
+	1    6950 3900
+	0    1    1    0
+$EndComp
+$Comp
+L R R?
+U 1 1 5BBD8E02
+P 7500 4150
+F 0 "R?" V 7580 4150 50  0000 C CNN
+F 1 "12k" V 7500 4150 50  0000 C CNN
+F 2 "" V 7430 4150 50  0001 C CNN
+F 3 "" H 7500 4150 50  0001 C CNN
+	1    7500 4150
+	1    0    0    -1
+$EndComp
+$Comp
+L Q_NPN_BCE Q?
+U 1 1 5BBD8F34
+P 7800 3200
+F 0 "Q?" H 8000 3250 50  0000 L CNN
+F 1 "TIP35" H 8000 3150 50  0000 L CNN
+F 2 "" H 8000 3300 50  0001 C CNN
+F 3 "" H 7800 3200 50  0001 C CNN
+	1    7800 3200
+	0    -1   -1   0
+$EndComp
+$Comp
+L Q_NPN_ECB Q?
+U 1 1 5BBD90A4
+P 7500 3600
+F 0 "Q?" H 7700 3650 50  0000 L CNN
+F 1 "BD139" H 7700 3550 50  0000 L CNN
+F 2 "" H 7700 3700 50  0001 C CNN
+F 3 "" H 7500 3600 50  0001 C CNN
+	1    7500 3600
+	0    -1   -1   0
+$EndComp
+Connection ~ 5000 4100
+Wire Wire Line
+	5800 4200 5800 4400
+Wire Wire Line
+	5000 4100 4900 4100
+Wire Wire Line
+	5000 4000 5000 4400
+Wire Wire Line
+	4900 4000 5000 4000
+Wire Wire Line
+	4900 3900 5500 3900
+Wire Wire Line
+	5000 4400 8400 4400
+Wire Wire Line
+	5300 4300 5300 4500
+Wire Wire Line
+	5300 4000 5300 3900
+Connection ~ 5300 3900
+Connection ~ 5300 4400
+Wire Wire Line
+	6100 3900 6300 3900
+Wire Wire Line
+	6200 3100 6200 4000
+Connection ~ 6200 3900
+Wire Wire Line
+	6600 3900 6800 3900
+Wire Wire Line
+	6700 4000 6700 3900
+Connection ~ 6700 3900
+Wire Wire Line
+	7100 3900 7500 3900
+Wire Wire Line
+	7200 3900 7200 4000
+Wire Wire Line
+	7500 3800 7500 4000
+Connection ~ 7200 3900
+Wire Wire Line
+	7500 4400 7500 4300
+Connection ~ 5800 4400
+Wire Wire Line
+	6200 4300 6200 4400
+Connection ~ 6200 4400
+Wire Wire Line
+	6700 4400 6700 4300
+Connection ~ 6700 4400
+Wire Wire Line
+	7200 4400 7200 4300
+Connection ~ 7200 4400
+Connection ~ 7500 3900
+Wire Wire Line
+	7700 3500 7800 3500
+Wire Wire Line
+	7800 3500 7800 3400
+Wire Wire Line
+	7600 3100 6200 3100
+Wire Wire Line
+	7300 3500 7200 3500
+Wire Wire Line
+	7200 3500 7200 3100
+Connection ~ 7200 3100
+Wire Wire Line
+	8000 3100 8400 3100
+Connection ~ 7500 4400
+$Comp
+L R R?
+U 1 1 5BBD94BE
+P 8100 3750
+F 0 "R?" V 8180 3750 50  0000 C CNN
+F 1 "330" V 8100 3750 50  0000 C CNN
+F 2 "" V 8030 3750 50  0001 C CNN
+F 3 "" H 8100 3750 50  0001 C CNN
+	1    8100 3750
+	1    0    0    -1
+$EndComp
+$Comp
+L LED D?
+U 1 1 5BBD95B9
+P 8100 4150
+F 0 "D?" H 8100 4250 50  0000 C CNN
+F 1 "LED" H 8100 4050 50  0000 C CNN
+F 2 "" H 8100 4150 50  0001 C CNN
+F 3 "" H 8100 4150 50  0001 C CNN
+	1    8100 4150
+	0    -1   -1   0
+$EndComp
+Wire Wire Line
+	8100 4000 8100 3900
+Wire Wire Line
+	8100 3100 8100 3600
+Connection ~ 8100 3100
+Wire Wire Line
+	8100 4300 8100 4400
+Connection ~ 8100 4400
+Wire Wire Line
+	8400 3100 8400 3800
+Wire Wire Line
+	8400 3800 8600 3800
+Wire Wire Line
+	8600 3900 8400 3900
+Wire Wire Line
+	8400 3900 8400 4400
 $EndSCHEMATC
